File: B3PKey.sch (KiCad schematic (older format))
At the start: 178 parts, among them SW1 SW_Push, U1 ATmega32U4-AU, Y1 16MHz

Commit message: Update layout
Parts:
- MX74: footprint MX_Only:MXOnly-3U-ReversedStabilizers-NoLED -> MX_Only:MXOnly-2U-ReversedStabilizers-NoLED
- MX75: footprint MX_Only:MXOnly-1U-NoLED -> MX_Only:MXOnly-2U-ReversedStabilizers-NoLED
Connections:
- net COL6: now also MX75.1 (COL)
- net COL7: no longer MX75.1 (COL)
Other:
- moved on the sheet: D75, MX75
Changed lines of the file:
@@
 	11950 7600 11950 7700
-$Comp
-L MX_Alps_Hybrid:MX-NoLED MX80
-U 1 1 603888A2
-P 13100 7250
-F 0 "MX80" H 13133 7473 60  0000 C CNN
-F 1 "MX-NoLED" H 13133 7399 20  0000 C CNN
-F 2 "MX_Only:MXOnly-1U-NoLED" H 12475 7225 60  0001 C CNN
-F 3 "" H 12475 7225 60  0001 C CNN
-	1    13100 7250
-	1    0    0    -1
-$EndComp
 $Comp
 L Device:D_Small D79
@@
 	11400 7600 11400 7700
 $Comp
-L MX_Alps_Hybrid:MX-NoLED MX79
-U 1 1 6038888E
-P 12550 7250
-F 0 "MX79" H 12583 7473 60  0000 C CNN
-F 1 "MX-NoLED" H 12583 7399 20  0000 C CNN
-F 2 "MX_Only:MXOnly-1U-NoLED" H 11925 7225 60  0001 C CNN
-F 3 "" H 11925 7225 60  0001 C CNN
-	1    12550 7250
-	1    0    0    -1
-$EndComp
-$Comp
 L Device:D_Small D78
 U 1 1 60388888
@@
 	10850 7600 10850 7700
 $Comp
-L MX_Alps_Hybrid:MX-NoLED MX78
-U 1 1 60388881
-P 12000 7250
-F 0 "MX78" H 12033 7473 60  0000 C CNN
-F 1 "MX-NoLED" H 12033 7399 20  0000 C CNN
-F 2 "MX_Only:MXOnly-1U-NoLED" H 11375 7225 60  0001 C CNN
-F 3 "" H 11375 7225 60  0001 C CNN
-	1    12000 7250
-	1    0    0    -1
-$EndComp
-$Comp
 L Device:D_Small D77
 U 1 1 60388878
@@
 $EndComp
 $Comp
-L MX_Alps_Hybrid:MX-NoLED MX77
-U 1 1 60388871
-P 11450 7250
-F 0 "MX77" H 11483 7473 60  0000 C CNN
-F 1 "MX-NoLED" H 11483 7399 20  0000 C CNN
-F 2 "MX_Only:MXOnly-1U-NoLED" H 10825 7225 60  0001 C CNN
-F 3 "" H 10825 7225 60  0001 C CNN
-	1    11450 7250
-	1    0    0    -1
-$EndComp
-$Comp
 L Device:D_Small D76
 U 1 1 6038886B
@@
 $EndComp
 $Comp
-L MX_Alps_Hybrid:MX-NoLED MX76
-U 1 1 60388864
-P 10900 7250
-F 0 "MX76" H 10933 7473 60  0000 C CNN
-F 1 "MX-NoLED" H 10933 7399 20  0000 C CNN
-F 2 "MX_Only:MXOnly-1U-NoLED" H 10275 7225 60  0001 C CNN
-F 3 "" H 10275 7225 60  0001 C CNN
-	1    10900 7250
-	1    0    0    -1
-$EndComp
-$Comp
 L Device:D_Small D75
 U 1 1 6038885B
-P 10300 7500
-F 0 "D75" H 10300 7600 50  0000 R CNN
-F 1 "D_Small" H 10650 7600 50  0000 R CNN
-F 2 "Diode_SMD:D_SOD-123" V 10300 7500 50  0001 C CNN
-F 3 "~" V 10300 7500 50  0001 C CNN
-	1    10300 7500
+P 9750 7500
+F 0 "D75" H 9750 7600 50  0000 R CNN
+F 1 "D_Small" H 10100 7600 50  0000 R CNN
+F 2 "Diode_SMD:D_SOD-123" V 9750 7500 50  0001 C CNN
+F 3 "~" V 9750 7500 50  0001 C CNN
+	1    9750 7500
 	0    -1   -1   0
 $EndComp
@@
 F 0 "MX74" H 9283 7473 60  0000 C CNN
 F 1 "MX-NoLED" H 9283 7399 20  0000 C CNN
-F 2 "MX_Only:MXOnly-3U-ReversedStabilizers-NoLED" H 8625 7225 60  0001 C CNN
+F 2 "MX_Only:MXOnly-2U-ReversedStabilizers-NoLED" H 8625 7225 60  0001 C CNN
 F 3 "" H 8625 7225 60  0001 C CNN
 	1    9250 7250
@@
 F 3 "" H 10275 4675 60  0001 C CNN
 	1    10900 4700
-	1    0    0    -1
-$EndComp
-$Comp
-L MX_Alps_Hybrid:MX-NoLED MX75
-U 1 1 60388854
-P 10350 7250
-F 0 "MX75" H 10383 7473 60  0000 C CNN
-F 1 "MX-NoLED" H 10383 7399 20  0000 C CNN
-F 2 "MX_Only:MXOnly-1U-NoLED" H 9725 7225 60  0001 C CNN
-F 3 "" H 9725 7225 60  0001 C CNN
-	1    10350 7250
 	1    0    0    -1
 $EndComp
@@
 Wire Wire Line
 	8100 7700 9200 7700
-Wire Wire Line
-	9200 7700 10300 7700
 $Comp
 L Device:D_Small D81
@@
 	1    0    0    -1
 $EndComp
-Wire Wire Line
-	10500 6350 10500 7200
-Connection ~ 10500 6350
-Wire Wire Line
-	10300 7600 10300 7700
-Connection ~ 10300 7700
-Wire Wire Line
-	10300 7700 10850 7700
+$Comp
+L MX_Alps_Hybrid:MX-NoLED MX75
+U 1 1 60388854
+P 9800 7250
+F 0 "MX75" H 9833 7473 60  0000 C CNN
+F 1 "MX-NoLED" H 9833 7399 20  0000 C CNN
+F 2 "MX_Only:MXOnly-2U-ReversedStabilizers-NoLED" H 9175 7225 60  0001 C CNN
+F 3 "" H 9175 7225 60  0001 C CNN
+	1    9800 7250
+	1    0    0    -1
+$EndComp
+$Comp
+L MX_Alps_Hybrid:MX-NoLED MX76
+U 1 1 60388864
+P 10900 7250
+F 0 "MX76" H 10933 7473 60  0000 C CNN
+F 1 "MX-NoLED" H 10933 7399 20  0000 C CNN
+F 2 "MX_Only:MXOnly-1U-NoLED" H 10275 7225 60  0001 C CNN
+F 3 "" H 10275 7225 60  0001 C CNN
+	1    10900 7250
+	1    0    0    -1
+$EndComp
+$Comp
+L MX_Alps_Hybrid:MX-NoLED MX77
+U 1 1 60388871
+P 11450 7250
+F 0 "MX77" H 11483 7473 60  0000 C CNN
+F 1 "MX-NoLED" H 11483 7399 20  0000 C CNN
+F 2 "MX_Only:MXOnly-1U-NoLED" H 10825 7225 60  0001 C CNN
+F 3 "" H 10825 7225 60  0001 C CNN
+	1    11450 7250
+	1    0    0    -1
+$EndComp
+$Comp
+L MX_Alps_Hybrid:MX-NoLED MX78
+U 1 1 60388881
+P 12000 7250
+F 0 "MX78" H 12033 7473 60  0000 C CNN
+F 1 "MX-NoLED" H 12033 7399 20  0000 C CNN
+F 2 "MX_Only:MXOnly-1U-NoLED" H 11375 7225 60  0001 C CNN
+F 3 "" H 11375 7225 60  0001 C CNN
+	1    12000 7250
+	1    0    0    -1
+$EndComp
+$Comp
+L MX_Alps_Hybrid:MX-NoLED MX79
+U 1 1 6038888E
+P 12550 7250
+F 0 "MX79" H 12583 7473 60  0000 C CNN
+F 1 "MX-NoLED" H 12583 7399 20  0000 C CNN
+F 2 "MX_Only:MXOnly-1U-NoLED" H 11925 7225 60  0001 C CNN
+F 3 "" H 11925 7225 60  0001 C CNN
+	1    12550 7250
+	1    0    0    -1
+$EndComp
+$Comp
+L MX_Alps_Hybrid:MX-NoLED MX80
+U 1 1 603888A2
+P 13100 7250
+F 0 "MX80" H 13133 7473 60  0000 C CNN
+F 1 "MX-NoLED" H 13133 7399 20  0000 C CNN
+F 2 "MX_Only:MXOnly-1U-NoLED" H 12475 7225 60  0001 C CNN
+F 3 "" H 12475 7225 60  0001 C CNN
+	1    13100 7250
+	1    0    0    -1
+$EndComp
+Wire Wire Line
+	9200 7700 9750 7700
+Wire Wire Line
+	9950 6350 9950 7200
+Connection ~ 9950 6350
+Wire Wire Line
+	9750 7600 9750 7700
+Connection ~ 9750 7700
+Wire Wire Line
+	9750 7700 10850 7700
 $EndSCHEMATC

Commit message: Route USB traces
Connections:
- net D_N: now reaches R3.1, U1.3 (D-)
- net D_P: now reaches R2.1, U1.4 (D+)
Changed lines of the file:
@@
 Wire Wire Line
 	9750 7700 10850 7700
+Text Label 2050 8500 0    50   ~ 0
+D_P
+Text Label 2050 8600 0    50   ~ 0
+D_N
 $EndSCHEMATC
