File: B3PKey.kicad_pcb (KiCad board)
At the start: 2 copper layers, 265.7 x 115.3 mm, 175 parts, among them SW1 SW_Push, U1 ATmega32U4-AU, Y1 16MHz

Commit message: Update Gerbers
Parts:
- removed REF**: D_DO-35_SOD27_P7.62mm_Horizontal, Diode_THT:D_DO-35_SOD27_P7.62mm_Horizontal
Changed lines of the file:
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@@
     (tracks 731)
     (zones 0)
-    (modules 175)
+    (modules 174)
     (nets 121)
   )
@@
     (add_net VCC)
   )
-  (module Diode_THT:D_DO-35_SOD27_P7.62mm_Horizontal (layer F.Cu)
-    (at 192.151 197.104)
-    (descr "Diode, DO-35_SOD27 series, Axial, Horizontal, pin pitch=7.62mm, , length*diameter=4*2mm^2, , http://www.diodes.com/_files/packages/DO-35.pdf")
-    (tags "Diode DO-35_SOD27 series Axial Horizontal pin pitch 7.62mm  length 4mm diameter 2mm")
-    (fp_text reference REF** (at 3.81 -2.12) (layer F.SilkS)
-      (effects (font (size 1 1) (thickness 0.15)))
-    )
-    (fp_text value D_DO-35_SOD27_P7.62mm_Horizontal (at 3.81 2.12) (layer F.Fab)
-      (effects (font (size 1 1) (thickness 0.15)))
-    )
-    (fp_text user K (at 0 -1.8) (layer F.SilkS)
-      (effects (font (size 1 1) (thickness 0.15)))
-    )
-    (fp_text user K (at 0 -1.8) (layer F.Fab)
-      (effects (font (size 1 1) (thickness 0.15)))
-    )
-    (fp_text user %R (at 4.11 0) (layer F.Fab)
-      (effects (font (size 0.8 0.8) (thickness 0.12)))
-    )
-    (fp_line (start 8.67 -1.25) (end -1.05 -1.25) (layer F.CrtYd) (width 0.05))
-    (fp_line (start 8.67 1.25) (end 8.67 -1.25) (layer F.CrtYd) (width 0.05))
-    (fp_line (start -1.05 1.25) (end 8.67 1.25) (layer F.CrtYd) (width 0.05))
-    (fp_line (start -1.05 -1.25) (end -1.05 1.25) (layer F.CrtYd) (width 0.05))
-    (fp_line (start 2.29 -1.12) (end 2.29 1.12) (layer F.SilkS) (width 0.12))
-    (fp_line (start 2.53 -1.12) (end 2.53 1.12) (layer F.SilkS) (width 0.12))
-    (fp_line (start 2.41 -1.12) (end 2.41 1.12) (layer F.SilkS) (width 0.12))
-    (fp_line (start 6.58 0) (end 5.93 0) (layer F.SilkS) (width 0.12))
-    (fp_line (start 1.04 0) (end 1.69 0) (layer F.SilkS) (width 0.12))
-    (fp_line (start 5.93 -1.12) (end 1.69 -1.12) (layer F.SilkS) (width 0.12))
-    (fp_line (start 5.93 1.12) (end 5.93 -1.12) (layer F.SilkS) (width 0.12))
-    (fp_line (start 1.69 1.12) (end 5.93 1.12) (layer F.SilkS) (width 0.12))
-    (fp_line (start 1.69 -1.12) (end 1.69 1.12) (layer F.SilkS) (width 0.12))
-    (fp_line (start 2.31 -1) (end 2.31 1) (layer F.Fab) (width 0.1))
-    (fp_line (start 2.51 -1) (end 2.51 1) (layer F.Fab) (width 0.1))
-    (fp_line (start 2.41 -1) (end 2.41 1) (layer F.Fab) (width 0.1))
-    (fp_line (start 7.62 0) (end 5.81 0) (layer F.Fab) (width 0.1))
-    (fp_line (start 0 0) (end 1.81 0) (layer F.Fab) (width 0.1))
-    (fp_line (start 5.81 -1) (end 1.81 -1) (layer F.Fab) (width 0.1))
-    (fp_line (start 5.81 1) (end 5.81 -1) (layer F.Fab) (width 0.1))
-    (fp_line (start 1.81 1) (end 5.81 1) (layer F.Fab) (width 0.1))
-    (fp_line (start 1.81 -1) (end 1.81 1) (layer F.Fab) (width 0.1))
-    (pad 2 thru_hole oval (at 7.62 0) (size 1.6 1.6) (drill 0.8) (layers *.Cu *.Mask))
-    (pad 1 thru_hole rect (at 0 0) (size 1.6 1.6) (drill 0.8) (layers *.Cu *.Mask))
-    (model ${KISYS3DMOD}/Diode_THT.3dshapes/D_DO-35_SOD27_P7.62mm_Horizontal.wrl
-      (at (xyz 0 0 0))
-      (scale (xyz 1 1 1))
-      (rotate (xyz 0 0 0))
-    )
-  )
   (module MX_Only:MXOnly-6U-Centered-ReversedStabilizers-NoLED (layer F.Cu)

Commit message: Add silkscreen logo, update gerbers
Parts:
- added G***: LOGO, logo:logo3, B.Cu at (179.6, 182.4)

Commit message: Update silkscreen
Parts:
- moved G*** 2.13 mm to (178.9, 180.3)
Changed lines of the file:
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@@
   )
   (module logo:logo3 (layer B.Cu)
-    (at 179.578 182.372 180)
+    (at 178.943 180.34 180)
     (fp_text reference G*** (at 0 0) (layer B.SilkS) hide
       (effects (font (size 1.524 1.524) (thickness 0.3)) (justify mirror))
@@
     )
   )
-  (gr_line (start 169.206552 184.243042) (end 169.206552 186.148042) (layer B.SilkS) (width 0.12))
+  (gr_line (start 168.571552 182.211042) (end 168.571552 184.116042) (layer B.SilkS) (width 0.12))
   (gr_arc (start 81.901349 81.899999) (end 81.901349 79.899999) (angle -90) (layer Edge.Cuts) (width 0.2))
   (gr_line (start 102.87 77.899999) (end 102.87 79.899999) (layer Edge.Cuts) (width 0.2))
@@
   (gr_arc (start 81.901349 191.15016) (end 79.901349 191.15016) (angle -90) (layer Edge.Cuts) (width 0.2))
   (gr_line (start 343.5517 193.15016) (end 81.90135 193.15016) (layer Edge.Cuts) (width 0.2))
-  (gr_line (start 161.840552 186.148043) (end 162.348552 186.148042) (layer B.SilkS) (width 0.12))
-  (gr_line (start 161.840552 184.243042) (end 161.840552 186.148043) (layer B.SilkS) (width 0.12))
-  (gr_line (start 169.206552 184.243042) (end 161.840552 184.243042) (layer B.SilkS) (width 0.12))
-  (gr_line (start 169.206552 186.148042) (end 163.237552 186.148042) (layer B.SilkS) (width 0.12))
-  (gr_text B3PKey (at 165.650552 185.259042) (layer B.SilkS)
+  (gr_line (start 161.205552 184.116043) (end 161.713552 184.116042) (layer B.SilkS) (width 0.12))
+  (gr_line (start 161.205552 182.211042) (end 161.205552 184.116043) (layer B.SilkS) (width 0.12))
+  (gr_line (start 168.571552 182.211042) (end 161.205552 182.211042) (layer B.SilkS) (width 0.12))
+  (gr_line (start 168.571552 184.116042) (end 162.602552 184.116042) (layer B.SilkS) (width 0.12))
+  (gr_text B3PKey (at 165.015552 183.227042) (layer B.SilkS)
     (effects (font (size 1.27 1.27) (thickness 0.254)) (justify mirror))
   )
-  (gr_line (start 176.655332 183.641309) (end 161.415332 183.641308) (layer B.SilkS) (width 0.12))
-  (gr_line (start 176.655332 181.228308) (end 176.655332 183.641309) (layer B.SilkS) (width 0.12))
-  (gr_line (start 154.557331 183.641309) (end 160.653332 183.641309) (layer B.SilkS) (width 0.12))
-  (gr_line (start 154.557331 181.228308) (end 154.557331 183.641309) (layer B.SilkS) (width 0.12))
-  (gr_line (start 176.655332 181.228308) (end 154.557331 181.228308) (layer B.SilkS) (width 0.12))
-  (gr_text "Elsbree Enterprises" (at 165.606332 182.498309) (layer B.SilkS)
+  (gr_line (start 176.020332 181.609309) (end 160.780332 181.609308) (layer B.SilkS) (width 0.12))
+  (gr_line (start 176.020332 179.196308) (end 176.020332 181.609309) (layer B.SilkS) (width 0.12))
+  (gr_line (start 153.922331 181.609309) (end 160.018332 181.609309) (layer B.SilkS) (width 0.12))
+  (gr_line (start 153.922331 179.196308) (end 153.922331 181.609309) (layer B.SilkS) (width 0.12))
+  (gr_line (start 176.020332 179.196308) (end 153.922331 179.196308) (layer B.SilkS) (width 0.12))
+  (gr_text "Elsbree Enterprises" (at 164.971332 180.466309) (layer B.SilkS)
     (effects (font (size 1.5 1.5) (thickness 0.3)) (justify mirror))
   )

Commit message: Update pbc outline, small tweaks
Also generate new gerbers and add case_open dxf file
Parts:
- C1, C2: value 30pF -> 22pF
- MX73: footprint MX_Only:MXOnly-6U-Centered-ReversedStabilizers-NoLED -> MX_Only:MXOnly-6U-ReversedStabilizers-NoLED
- moved R5 9.72 mm to (104.4, 81.5)
- moved R6 9.72 mm to (104.4, 83.6)
- moved D73 9.53 mm to (206.4, 188.9)
- moved F1 8.65 mm to (95.4, 83.6)
- moved R2 8.65 mm to (99.4, 83.6)
- moved R3 8.65 mm to (97.4, 83.6)
- moved USB1 6.56 mm to (98.4, 71.4)
- moved R4 1.53 mm to (219.9, 182.6), turned to 315 degrees
Connections:
- MX73 pad 1: COL5 -> COL6
Routing:
- net COL6: track 113.6 -> 128.7 mm
- net COL2: track 214.8 -> 204.8 mm
- net COL0: track 255.5 -> 245.5 mm
- net COL1: track 235.1 -> 225.1 mm
- net COL5: track 145.0 -> 135.6 mm, vias 2 -> 1
- net +5V: track 283.3 -> 292.4 mm
- net /D_P: track 217.1 -> 224.1 mm
- net /D_N: track 216.5 -> 223.5 mm
- net ROW1: track 326.4 -> 323.5 mm, vias 3 -> 2
- net D+: track 9.30 -> 7.13 mm
- net D-: track 9.64 -> 7.69 mm
- net /CC2: track 6.19 -> 4.93 mm
- net Net-(R4-Pad2): track 1.75 -> 2.86 mm
- net /CC1: track 10.6 -> 9.52 mm
- net VCC: track 13.6 -> 12.7 mm
Other:
- board size 265.7 x 115.3 mm -> 282.7 x 130.3 mm
- net class Power: trace_width 0.381 -> 0.508

Commit message: Update gerbers and outline
Other:
- board size 282.7 x 130.3 mm -> 265.7 x 121.8 mm
